Commit message: fixed bug

File: create3_urdf_assem_description/urdf/create3_urdf_assem.xacro (robot description, xacro)
@@ -65,7 +65,7 @@
 <link name="ArmLink_Assem_v2_1">
   <inertial>
-    <origin xyz="-0.0005551221331234757 -0.02678554127174524 0.03869458338113388" rpy="0 0 0"/>
+    <origin xyz="-0.0005551221331234618 -0.02678554127174529 0.03869458338113407" rpy="0 0 0"/>
     <mass value="0.130177049170526"/>
-    <inertia ixx="0.000222170706605568" iyy="0.000197795129567611" izz="3.658812708562e-05" ixy="-1.61004432074186e-09" iyz="-1.8967903760383e-07" ixz="2.24911220115609e-06"/>
+    <inertia ixx="0.000222170706605569" iyy="0.000197795129567611" izz="3.65881270856202e-05" ixy="-1.61004432073848e-09" iyz="-1.89679037603826e-07" ixz="2.24911220115566e-06"/>
   </inertial>
   <visual>
@@ -85,7 +85,7 @@
 <link name="ArmLink_Assem_v2_2">
   <inertial>
-    <origin xyz="-0.0005551221331235173 -0.026785541271745025 0.038694600994638895" rpy="0 0 0"/>
+    <origin xyz="-0.0005551221331234896 -0.02678554127174507 0.03869460099463928" rpy="0 0 0"/>
     <mass value="0.130177049170526"/>
-    <inertia ixx="0.00022217070660557" iyy="0.000197795129567612" izz="3.65881270856204e-05" ixy="-1.61004432074398e-09" iyz="-1.89679037603877e-07" ixz="2.24911220115609e-06"/>
+    <inertia ixx="0.000222170706605573" iyy="0.000197795129567616" izz="3.65881270856191e-05" ixy="-1.61004432075245e-09" iyz="-1.8967903760388e-07" ixz="2.24911220115653e-06"/>
   </inertial>
   <visual>
@@ -125,7 +125,7 @@
 <link name="DrivenArm_v2_1">
   <inertial>
-    <origin xyz="0.0018673970936629036 -1.0280938773921111e-09 0.021529759537284032" rpy="0 0 0"/>
+    <origin xyz="0.0018673970936628759 -1.0280939259643684e-09 0.021529759537284532" rpy="0 0 0"/>
     <mass value="0.00854038789073064"/>
-    <inertia ixx="3.53704128751319e-06" iyy="3.70293575717461e-06" izz="4.60395655026163e-07" ixy="-8.090130263838438e-16" iyz="1.565001993557476e-13" ixz="-6.60995881882369e-08"/>
+    <inertia ixx="3.53704128751298e-06" iyy="3.70293575717483e-06" izz="4.60395655026082e-07" ixy="-8.090113323179493e-16" iyz="1.565001993557476e-13" ixz="-6.60995881881284e-08"/>
   </inertial>
   <visual>
@@ -145,7 +145,7 @@
 <link name="DriverArm_v2_1">
   <inertial>
-    <origin xyz="0.0018282857610038283 1.3368481251475883e-06 0.020586093564154473" rpy="0 0 0"/>
+    <origin xyz="0.001828285761003412 1.336848125067791e-06 0.020586093564155028" rpy="0 0 0"/>
     <mass value="0.00894442654078101"/>
-    <inertia ixx="3.72210504394539e-06" iyy="3.87544643711511e-06" izz="4.78096502262091e-07" ixy="-9.003251554115695e-12" iyz="-2.63898014097946e-10" ixz="-7.32275454850152e-08"/>
+    <inertia ixx="3.72210504394539e-06" iyy="3.87544643711468e-06" izz="4.78096502262146e-07" ixy="-9.003251557503826e-12" iyz="-2.63898014104722e-10" ixz="-7.32275454851236e-08"/>
   </inertial>
   <visual>
@@ -165,7 +165,7 @@
 <link name="FrontArmLeft_v2_1">
   <inertial>
-    <origin xyz="0.002212740648021183 -3.802814928692902e-07 0.03526507682589175" rpy="0 0 0"/>
+    <origin xyz="0.0022127406480213496 -3.802814929100562e-07 0.035265076825892305" rpy="0 0 0"/>
     <mass value="0.00440333324799871"/>
-    <inertia ixx="8.07103574171179e-07" iyy="1.10375934229598e-06" izz="3.21260210004977e-07" ixy="-1.591343321459754e-12" iyz="-3.303251162184440e-11" ixz="-2.29806381504567e-08"/>
+    <inertia ixx="8.07103574171179e-07" iyy="1.10375934229577e-06" izz="3.21260210004991e-07" ixy="-1.591343322730304e-12" iyz="-3.303251162353846e-11" ixz="-2.29806381504567e-08"/>
   </inertial>
   <visual>
@@ -185,7 +185,7 @@
 <link name="FrontArmRight_v2_1">
   <inertial>
-    <origin xyz="0.002212740648066369 5.340535291073131e-07 0.03526507682586799" rpy="0 0 0"/>
+    <origin xyz="0.0022127406480665357 5.340535290708839e-07 0.035265076825868436" rpy="0 0 0"/>
     <mass value="0.0044033332479868"/>
-    <inertia ixx="8.0710360417474e-07" iyy="1.10375934229121e-06" izz="3.21260240006003e-07" ixy="1.648360665830787e-12" iyz="3.289259880770836e-11" ixz="-2.29806381508903e-08"/>
+    <inertia ixx="8.07103604174306e-07" iyy="1.10375934229121e-06" izz="3.21260240005963e-07" ixy="1.648360665830787e-12" iyz="3.289259880940242e-11" ixz="-2.29806381508903e-08"/>
   </inertial>
   <visual>
@@ -205,7 +205,7 @@
 <link name="LeftPad_v2_1">
   <inertial>
-    <origin xyz="-0.014500135487571925 0.0022332025380023234 0.028341191588216408" rpy="0 0 0"/>
+    <origin xyz="-0.014500135487571841 0.002233202538002273 0.028341191588217074" rpy="0 0 0"/>
     <mass value="0.0152834385878526"/>
-    <inertia ixx="3.79296682396363e-06" iyy="5.38017343292181e-06" izz="2.59536641118426e-06" ixy="5.106430482995118e-13" iyz="-7.70848043957385e-07" ixz="-5.422499688850779e-12"/>
+    <inertia ixx="3.7929668239645e-06" iyy="5.38017343292355e-06" izz="2.59536641118415e-06" ixy="5.106430449113800e-13" iyz="-7.70848043957413e-07" ixz="-5.422499472010345e-12"/>
   </inertial>
   <visual>
@@ -225,7 +225,7 @@
 <link name="RightPad_v2_1">
   <inertial>
-    <origin xyz="-0.014500027644216151 -0.002233057301935279 0.028341187437789073" rpy="0 0 0"/>
+    <origin xyz="-0.014500027644216262 -0.002233057301935324 0.028341187437789628" rpy="0 0 0"/>
     <mass value="0.0152834381646124"/>
-    <inertia ixx="3.79296716121295e-06" iyy="5.38017329065194e-06" izz="2.59536675226613e-06" ixy="1.091684502399579e-12" iyz="7.7084682724775e-07" ixz="-5.974396324881504e-12"/>
+    <inertia ixx="3.79296716121122e-06" iyy="5.38017329065194e-06" izz="2.59536675226613e-06" ixy="1.091684495623316e-12" iyz="7.7084682724775e-07" ixz="-5.974396324881504e-12"/>
   </inertial>
   <visual>
@@ -245,7 +245,7 @@
 <link name="RDS3225_-_for_URDF_v5_1">
   <inertial>
-    <origin xyz="-7.433028170189537e-07 -0.02683132902450605 0.012322771916488007" rpy="0 0 0"/>
+    <origin xyz="-7.433028169634426e-07 -0.026831329024506096 0.012322771916488617" rpy="0 0 0"/>
     <mass value="0.0791893057217848"/>
-    <inertia ixx="2.82106812690194e-05" iyy="1.58164077691415e-05" izz="1.74398753985518e-05" ixy="2.415999720201076e-11" iyz="4.12347903638339e-07" ixz="-5.356776740933489e-11"/>
+    <inertia ixx="2.82106812690159e-05" iyy="1.58164077691345e-05" izz="1.74398753985518e-05" ixy="2.415999719629328e-11" iyz="4.12347903638314e-07" ixz="-5.356776524093054e-11"/>
   </inertial>
   <visual>
@@ -265,7 +265,7 @@
 <link name="Base_v8_1">
   <inertial>
-    <origin xyz="0.00038555172899897017 0.002775906354052858 0.019181141479140074" rpy="0 0 0"/>
+    <origin xyz="0.0003855517289991367 0.0027759063540528173 0.01918114147914035" rpy="0 0 0"/>
     <mass value="0.172135511489978"/>
-    <inertia ixx="7.43707221079887e-05" iyy="7.65171561616304e-05" izz="0.000100049270469719" ixy="1.11277277933259e-07" iyz="2.44198108194339e-08" ixz="-5.13466019367876e-06"/>
+    <inertia ixx="7.43707221079887e-05" iyy="7.65171561616373e-05" izz="0.000100049270469717" ixy="1.11277277933266e-07" iyz="2.44198108193525e-08" ixz="-5.13466019367703e-06"/>
   </inertial>
   <visual>
